File: PCB/SimplePhotoFrame/SimplePhotoFrame.kicad_sch (KiCad schematic)
At the start: 32 parts, among them J1 Micro_SD_Card, J2 USB_C_Receptacle_PowerOnly_6P, SW1 SW_MEC_5G, SW2 SW_MEC_5G, SW3 SW_MEC_5G, SW4 SW_MEC_5G, SW5 SW_MEC_5G, SW6 SW_MEC_5G

Commit message: Updated
Other:
- note added: "DAT0(DO) - MISO CMD(DI) - MOSI"
Changed lines of the file:
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@@
 		(company "Takayuki Hara")
+	)
+	(text "DAT0(DO) - MISO\nCMD(DI) - MOSI"
+		(exclude_from_sim no)
+		(at 231.902 144.272 0)
+		(effects
+			(font
+				(size 1.27 1.27)
+			)
+		)
 	)
 	(text "L で点灯\nH で消灯\nLEDx は、FPGA内PullUp"
